File: mg/mg.kicad_sch (KiCad schematic)
At the start: 35 parts, among them IC1 LM393D, U1 LMH6645MFX_NOPB, U2 LMV7219M7_NOPB, U6 SN74LV123ARGYRG4, Y1 ACOUSTIC RX

Commit message: Fully reverse engineered. Added comments to schematic.
Parts:
- renumbered IC1 to U1
Other:
- sheet PLL VCO ports: added TEST; removed VCO_OUT
- note added: "150 KHz high pass filter"
- note added: "Blocks DC from 2V5 at input"
- note added: "Puillup"
- note added: "Sets gain"
- note added: "Sets one-shot durations"
- note added: "Supply voltage reference"
- note added: "bypass"
- note removed: "PIN2 may be measuring supply voltage (+5V)"
- note removed: "PULL UP"
- note removed: "low pass filter"
- moved on the sheet: R24
Changed lines of the file:
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@@
 (kicad_sch (version 20230409) (generator eeschema)
   (paper "A4")
-  (junction (at 124.46 121.92) (diameter 0) (color 0 0 0 0)
+  (junction (at 118.11 121.92) (diameter 0) (color 0 0 0 0)
   )
   (junction (at 161.29 123.19) (diameter 0) (color 0 0 0 0)
@@
     (stroke (width 0) (type default))
   )
-  (wire (pts (xy 124.46 139.7) (xy 124.46 129.54))
+  (wire (pts (xy 118.11 139.7) (xy 118.11 135.89))
     (stroke (width 0) (type default))
   )
@@
     (stroke (width 0) (type default))
   )
+  (wire (pts (xy 118.11 128.27) (xy 118.11 121.92))
+    (stroke (width 0) (type default))
+  )
   (wire (pts (xy 39.37 115.57) (xy 39.37 109.22))
     (stroke (width 0) (type default))
@@
     (stroke (width 0) (type default))
   )
-  (wire (pts (xy 118.11 121.92) (xy 124.46 121.92))
-    (stroke (width 0) (type default))
-  )
   (wire (pts (xy 140.97 80.01) (xy 146.05 80.01))
     (stroke (width 0) (type default))
@@
     (stroke (width 0) (type default))
   )
+  (wire (pts (xy 208.28 142.24) (xy 226.06 142.24))
+    (stroke (width 0) (type default))
+  )
   (wire (pts (xy 147.32 101.6) (xy 147.32 109.22))
     (stroke (width 0) (type default))
@@
     (stroke (width 0) (type default))
   )
-  (wire (pts (xy 124.46 121.92) (xy 133.35 121.92))
+  (wire (pts (xy 118.11 121.92) (xy 133.35 121.92))
     (stroke (width 0) (type default))
   )
@@
   (wire (pts (xy 208.28 54.61) (xy 212.09 54.61))
     (stroke (width 0) (type default))
+  )
+  (rectangle (start 104.14 113.03) (end 128.27 148.59)
+    (stroke (width 0) (type default))
+    (fill (type none))
   )
   (rectangle (start 88.9 170.18) (end 102.87 184.15)
@@
     (effects (font (size 1.27 1.27)) (justify left bottom))
   )
+  (text "Supply\nvoltage\nreference" (exclude_from_sim no)
+ (at 83.82 30.48 0)
+    (effects (font (size 1.27 1.27)) (justify left bottom))
+  )
   (text "Dual one-shot. /A is not used.\n#1 maintains OUTPUT high for a minimum time\nR_ext / C_ext and C_ext set duration.\n\n" (exclude_from_sim no)
     (at 205.74 113.03 0)
     (effects (font (size 1.27 1.27)) (justify left bottom))
   )
+  (text "bypass" (exclude_from_sim no)
+ (at 245.11 77.47 0)
+    (effects (font (size 1.27 1.27)) (justify left bottom))
+  )
   (text "C14 is a\nshared bypass" (exclude_from_sim no)
  (at 86.36 160.02 0)
     (effects (font (size 1.27 1.27)) (justify left bottom))
   )
+  (text "Sets one-shot\ndurations" (exclude_from_sim no)
+ (at 185.42 43.18 0)
+    (effects (font (size 1.27 1.27)) (justify left bottom))
+  )
   (text "DUAL COMPARATOR" (exclude_from_sim no)
  (at 24.13 21.59 0)
     (effects (font (size 1.27 1.27)) (justify left bottom))
   )
+  (text "Sets gain" (exclude_from_sim no)
+ (at 100.33 167.64 0)
+    (effects (font (size 1.27 1.27)) (justify left bottom))
+  )
   (text "478 mV" (exclude_from_sim no)
  (at 91.44 49.53 0)
     (effects (font (size 1.27 1.27)) (justify left bottom))
   )
-  (text "PULL UP" (exclude_from_sim no)
+  (text "Puillup" (exclude_from_sim no)
  (at 132.08 57.15 0)
     (effects (font (size 1.27 1.27)) (justify left bottom))
@@
     (effects (font (size 1.27 1.27)) (justify left bottom))
   )
-  (text "PIN2 may be measuring\nsupply voltage (+5V)" (exclude_from_sim no)
- (at -24.13 39.37 0)
+  (text "150 KHz\nhigh pass\nfilter" (exclude_from_sim no)
+ (at 104.14 113.03 0)
+    (effects (font (size 1.27 1.27)) (justify left bottom))
+  )
+  (text "Supply\nvoltage\nreference" (exclude_from_sim no)
+ (at 54.61 33.02 0)
     (effects (font (size 1.27 1.27)) (justify left bottom))
   )
@@
     (effects (font (size 1.27 1.27)) (justify left bottom))
   )
-  (text "low pass filter" (exclude_from_sim no)
+  (text "Blocks DC from 2V5 at input" (exclude_from_sim no)
  (at 104.14 179.07 0)
     (effects (font (size 1.27 1.27)) (justify left bottom))
@@
   (symbol (lib_name "LM393D_1") (lib_id "SamacSys_Parts:LM393D") (at 43.18 58.42 0) (unit 1)
     (in_bom yes) (on_board yes) (dnp no) (fields_autoplaced)
-    (property "Reference" "IC1" (at 49.53 54.61 0)
-      (effects (font (size 1.27 1.27)))
-    )
-    (property "Value" "LM393D" (at 62.23 76.2 0)
-      (effects (font (size 1.27 1.27)))
+    (property "Reference" "U1" (at 59.3441 50.8 0)
+      (effects (font (size 1.27 1.27)) (justify left))
+    )
+    (property "Value" "LM393D" (at 59.3441 53.34 0)
+      (effects (font (size 1.27 1.27)) (justify left))
     )
     (property "Footprint" "SOIC127P600X175-8N" (at 67.31 153.34 0)
@@
       (project "mg"
         (path "/3b629f3b-e9cd-474a-b8e0-426e6f380223"
-          (reference "IC1") (unit 1)
-        )
-      )
-    )
-  )
-  (symbol (lib_id "power:GND") (at 124.46 139.7 0) (unit 1)
+          (reference "U1") (unit 1)
+        )
+      )
+    )
+  )
+  (symbol (lib_id "power:GND") (at 118.11 139.7 0) (unit 1)
     (in_bom yes) (on_board yes) (dnp no) (fields_autoplaced)
-    (property "Reference" "#PWR012" (at 124.46 146.05 0)
-      (effects (font (size 1.27 1.27)) hide)
-    )
-    (property "Value" "GND" (at 124.46 144.78 0)
-      (effects (font (size 1.27 1.27)))
-    )
-    (property "Footprint" "" (at 124.46 139.7 0)
-      (effects (font (size 1.27 1.27)) hide)
-    )
-    (property "Datasheet" "" (at 124.46 139.7 0)
+    (property "Reference" "#PWR012" (at 118.11 146.05 0)
+      (effects (font (size 1.27 1.27)) hide)
+    )
+    (property "Value" "GND" (at 118.11 144.78 0)
+      (effects (font (size 1.27 1.27)))
+    )
+    (property "Footprint" "" (at 118.11 139.7 0)
+      (effects (font (size 1.27 1.27)) hide)
+    )
+    (property "Datasheet" "" (at 118.11 139.7 0)
       (effects (font (size 1.27 1.27)) hide)
     )
@@
     )
   )
-  (symbol (lib_id "Device:R") (at 124.46 125.73 180) (unit 1)
-    (in_bom yes) (on_board yes) (dnp no)
-    (property "Reference" "R24" (at 123.19 124.46 0)
-      (effects (font (size 1.27 1.27)) (justify left))
-    )
-    (property "Value" "6K8" (at 123.19 127 0)
-      (effects (font (size 1.27 1.27)) (justify left))
-    )
-    (property "Footprint" "mg_footprints:C_0603Metric" (at 126.238 125.73 90)
-      (effects (font (size 1.27 1.27)) hide)
-    )
-    (property "Datasheet" "~" (at 124.46 125.73 0)
+  (symbol (lib_id "Device:R") (at 118.11 132.08 180) (unit 1)
+    (in_bom yes) (on_board yes) (dnp no)
+    (property "Reference" "R24" (at 116.84 130.81 0)
+      (effects (font (size 1.27 1.27)) (justify left))
+    )
+    (property "Value" "6K8" (at 116.84 133.35 0)
+      (effects (font (size 1.27 1.27)) (justify left))
+    )
+    (property "Footprint" "mg_footprints:C_0603Metric" (at 119.888 132.08 90)
+      (effects (font (size 1.27 1.27)) hide)
+    )
+    (property "Datasheet" "~" (at 118.11 132.08 0)
       (effects (font (size 1.27 1.27)) hide)
     )
@@
     (instances
       (project "mg"
-        (path "/3b629f3b-e9cd-474a-b8e0-426e6f380223" (page "5"))
-      )
-    )
-  )
-  (sheet (at 325.12 72.39) (size 33.02 22.86) (fields_autoplaced)
+        (path "/3b629f3b-e9cd-474a-b8e0-426e6f380223" (page "3"))
+      )
+    )
+  )
+  (sheet (at 226.06 132.08) (size 33.02 15.24) (fields_autoplaced)
     (stroke (width 0.1524) (type solid))
     (fill (color 0 0 0 0.0000))
-    (property "Sheetname" "PLL VCO" (at 325.12 71.6784 0)
+    (property "Sheetname" "PLL VCO" (at 226.06 131.3684 0)
       (effects (font (size 1.27 1.27)) (justify left bottom))
     )
-    (property "Sheetfile" "pll-vco.kicad_sch" (at 325.12 95.8346 0)
+    (property "Sheetfile" "pll-vco.kicad_sch" (at 226.06 147.9046 0)
       (effects (font (size 1.27 1.27)) (justify left top))
     )
-    (pin "VCO_OUT" input (at 325.12 80.01 180)
-      (effects (font (size 1.27 1.27)) (justify left))
-    )
-    (instances
-      (project "mg"
-        (path "/3b629f3b-e9cd-474a-b8e0-426e6f380223" (page "3"))
-      )
-    )
+    (pin "TEST" input (at 226.06 142.24 180)
+      (effects (font (size 1.27 1.27)) (justify left))
+    )
+    (instances
+      (project "mg"
+        (path "/3b629f3b-e9cd-474a-b8e0-426e6f380223" (page "2"))
+      )
+    )
